File: PCB/Seed_xiao_nrf_kit_phone.kicad_sch (KiCad schematic)
At the start: 37 parts, among them J1 4pin header, Q2 AO3400A, SW1 TS-1187A-B-A-B, SW10 TS-1187A-B-A-B, SW11 TS-1187A-B-A-B, SW12 TS-1187A-B-A-B, SW2 TS-1187A-B-A-B, SW3 TS-1187A-B-A-B, SW4 TS-1187A-B-A-B, SW5 TS-1187A-B-A-B, SW6 TS-1187A-B-A-B, SW7 TS-1187A-B-A-B, SW8 TS-1187A-B-A-B, SW9 TS-1187A-B-A-B, U1 TCA8418RTWR, U2 XIAO-nRF52840-SMD, U6 BME280, U9 WIO-SX1262-DIP

Commit message: fixed XIAO showing on BOM &  POS
Parts:
- U2: now left out of the parts list
Changed lines of the file:
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@@
 		(body_style 1)
 		(exclude_from_sim no)
-		(in_bom yes)
+		(in_bom no)
 		(on_board yes)
-		(in_pos_files yes)
+		(in_pos_files no)
 		(dnp no)
 		(fields_autoplaced yes)
